File: board/WiFiLEDController_FET/WiFiLEDController_FET.kicad_pcb (KiCad board)
At the start: 2 copper layers, 80 x 50 mm, 40 parts, among them J1 12V_In, J2 Serial, J3 Conn_01x04_Female, Q1 IRLZ34N, Q2 IRLZ34N, Q3 IRLZ34N, SW1 Reset, SW2 Flash, U1 LM25011, U2 ESP-07

Commit message: Layout done
Parts:
- moved R1 0.64 mm to (187.3, 88.3)
Routing:
- net /G_Out: track 26.8 -> 53.5 mm
- net /B_Out: track 13.3 -> 26.6 mm
- net /R_Out: track 7.40 -> 14.8 mm
- net /PWM_G: track 46.0 -> 51.4 mm
- net +3V3: track 34.2 -> 37.0 mm
- net Net-(R1-Pad1): track 30.9 -> 32.0 mm
- net GND: vias 80 -> 113
Other:
- board text added: "4A Max. per Channel!"
- board text removed: "2A Max. per Channel!"

Commit message: Minor Layout Changes
Routing:
- net /12V_Out: track 76.5 -> 66.3 mm, vias 6 -> 13
- net /G_Out: track 53.5 -> 56.2 mm
- added copper zone on B.Cu, net /12V_Out
Changed lines of the file:
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@@
     (thickness 1.6)
     (drawings 14)
-    (tracks 346)
+    (tracks 337)
     (zones 0)
     (modules 40)
@@
   )
   (setup
-    (last_trace_width 2)
+    (last_trace_width 0.25)
     (user_trace_width 0.5)
     (user_trace_width 1)
@@
     (mod_text_size 1 1)
     (mod_text_width 0.15)
-    (pad_size 2.5 2.5)
-    (pad_drill 1.3)
+    (pad_size 1.7 1.7)
+    (pad_drill 1)
     (pad_to_mask_clearance 0.051)
     (solder_mask_min_width 0.25)
@@
     (fp_line (start -10.03 -1.27) (end -2.49 -1.27) (layer F.Fab) (width 0.1))
     (pad 4 thru_hole oval (at 0 7.62 180) (size 1.7 1.7) (drill 1) (layers *.Cu *.Mask)
-      (net 2 /12V_Out))
+      (net 2 /12V_Out) (zone_connect 2))
     (pad 3 thru_hole oval (at 0 5.08 180) (size 1.7 1.7) (drill 1) (layers *.Cu *.Mask)
       (net 16 /G_Out))
@@
   (segment (start 168.945 76.445) (end 166.37 76.445) (width 0.25) (layer F.Cu) (net 2) (status 20))
   (segment (start 169.05 76.34) (end 168.945 76.445) (width 0.25) (layer F.Cu) (net 2))
-  (segment (start 215.9 89.602919) (end 214.152499 87.855418) (width 2.5) (layer B.Cu) (net 2))
-  (segment (start 215.9 90.805) (end 215.9 89.602919) (width 2.5) (layer B.Cu) (net 2))
-  (segment (start 215.9 89.602919) (end 215.548541 89.251459) (width 2.5) (layer F.Cu) (net 2))
-  (segment (start 215.9 90.805) (end 215.9 89.602919) (width 2.5) (layer F.Cu) (net 2))
-  (segment (start 213.995 87.697919) (end 213.995 87.63) (width 2.5) (layer F.Cu) (net 2))
-  (segment (start 215.548541 89.251459) (end 215.421541 89.124459) (width 2.5) (layer F.Cu) (net 2))
-  (segment (start 214.596041 88.298959) (end 214.15154 87.85446) (width 2.5) (layer F.Cu) (net 2))
-  (segment (start 213.995 86.995) (end 213.995 86.36) (width 2.5) (layer F.Cu) (net 2))
-  (segment (start 213.995 85.725) (end 213.995 85.217) (width 2.5) (layer F.Cu) (net 2))
-  (segment (start 213.995 86.36) (end 213.995 86.106) (width 2.5) (layer F.Cu) (net 2))
-  (segment (start 213.995 87.63) (end 213.995 86.995) (width 2.5) (layer F.Cu) (net 2))
-  (segment (start 215.421541 89.124459) (end 214.786541 88.489459) (width 2.5) (layer F.Cu) (net 2))
-  (segment (start 214.786541 88.489459) (end 214.596041 88.298959) (width 2.5) (layer F.Cu) (net 2))
-  (via (at 214.786541 88.489459) (size 0.8) (drill 0.4) (layers F.Cu B.Cu) (net 2))
-  (segment (start 214.15154 87.85446) (end 213.995 87.697919) (width 2.5) (layer F.Cu) (net 2))
-  (segment (start 213.995 86.995) (end 213.995 86.995) (width 2.5) (layer F.Cu) (net 2))
-  (via (at 213.995 86.995) (size 0.8) (drill 0.4) (layers F.Cu B.Cu) (net 2))
-  (segment (start 213.995 86.106) (end 213.995 85.725) (width 2.5) (layer F.Cu) (net 2))
-  (segment (start 213.995 85.217) (end 213.995 85.09) (width 2.5) (layer F.Cu) (net 2))
-  (via (at 213.995 85.217) (size 0.8) (drill 0.4) (layers F.Cu B.Cu) (net 2))
   (segment (start 162.56 83.185) (end 161.29 81.915) (width 5) (layer B.Cu) (net 2))
   (segment (start 174.625 83.185) (end 162.56 83.185) (width 5) (layer B.Cu) (net 2))
+  (segment (start 214.152499 86.202501) (end 214.152499 86.202501) (width 5) (layer B.Cu) (net 2))
+  (segment (start 177.642501 86.202501) (end 174.625 83.185) (width 5) (layer B.Cu) (net 2))
   (segment (start 214.152499 86.202501) (end 177.642501 86.202501) (width 5) (layer B.Cu) (net 2))
-  (segment (start 177.642501 86.202501) (end 174.625 83.185) (width 5) (layer B.Cu) (net 2))
-  (via (at 215.421541 89.124459) (size 0.8) (drill 0.4) (layers F.Cu B.Cu) (net 2))
-  (via (at 214.15154 87.85446) (size 0.8) (drill 0.4) (layers F.Cu B.Cu) (net 2))
-  (via (at 213.995 86.106) (size 0.8) (drill 0.4) (layers F.Cu B.Cu) (net 2))
+  (via (at 213.487 85.979) (size 0.8) (drill 0.4) (layers F.Cu B.Cu) (net 2))
+  (via (at 216.281 87.63) (size 0.8) (drill 0.4) (layers F.Cu B.Cu) (net 2))
+  (via (at 214.884 87.63) (size 0.8) (drill 0.4) (layers F.Cu B.Cu) (net 2))
+  (via (at 214.884 84.455) (size 0.8) (drill 0.4) (layers F.Cu B.Cu) (net 2))
+  (via (at 216.281 84.455) (size 0.8) (drill 0.4) (layers F.Cu B.Cu) (net 2))
+  (via (at 214.884 85.979) (size 0.8) (drill 0.4) (layers F.Cu B.Cu) (net 2))
+  (via (at 213.487 84.455) (size 0.8) (drill 0.4) (layers F.Cu B.Cu) (net 2))
+  (via (at 213.487 87.63) (size 0.8) (drill 0.4) (layers F.Cu B.Cu) (net 2))
+  (via (at 213.487 89.408) (size 0.8) (drill 0.4) (layers F.Cu B.Cu) (net 2))
+  (via (at 216.281 85.979) (size 0.8) (drill 0.4) (layers F.Cu B.Cu) (net 2))
+  (via (at 214.884 89.408) (size 0.8) (drill 0.4) (layers F.Cu B.Cu) (net 2))
+  (via (at 216.281 89.408) (size 0.8) (drill 0.4) (layers F.Cu B.Cu) (net 2))
+  (via (at 213.487 91.186) (size 0.8) (drill 0.4) (layers F.Cu B.Cu) (net 2))
   (segment (start 167.885 79.645) (end 167.885 81.915) (width 0.25) (layer F.Cu) (net 3) (status 20))
   (segment (start 168.29 79.24) (end 167.885 79.645) (width 0.25) (layer F.Cu) (net 3))
@@
   (segment (start 215.9 95.885) (end 213.995 95.885) (width 2) (layer F.Cu) (net 15))
   (segment (start 213.995 95.885) (end 211.455 93.345) (width 2) (layer F.Cu) (net 15))
-  (segment (start 216.535 79.375) (end 209.55 79.375) (width 2) (layer B.Cu) (net 16))
-  (segment (start 220.98 83.82) (end 216.535 79.375) (width 2) (layer B.Cu) (net 16))
-  (segment (start 220.98 91.44) (end 220.98 83.82) (width 2) (layer B.Cu) (net 16))
+  (segment (start 219.075 93.345) (end 215.9 93.345) (width 2) (layer F.Cu) (net 16))
+  (segment (start 220.98 91.44) (end 219.075 93.345) (width 2) (layer F.Cu) (net 16))
+  (segment (start 220.98 81.534) (end 220.98 91.44) (width 2) (layer F.Cu) (net 16))
+  (segment (start 209.55 79.375) (end 218.821 79.375) (width 2) (layer F.Cu) (net 16))
+  (segment (start 218.821 79.375) (end 220.98 81.534) (width 2) (layer F.Cu) (net 16))
+  (segment (start 218.821 79.375) (end 209.55 79.375) (width 2) (layer B.Cu) (net 16))
+  (segment (start 220.98 81.534) (end 218.821 79.375) (width 2) (layer B.Cu) (net 16))
+  (segment (start 220.98 91.44) (end 220.98 81.534) (width 2) (layer B.Cu) (net 16))
   (segment (start 215.9 93.345) (end 219.075 93.345) (width 2) (layer B.Cu) (net 16))
   (segment (start 219.075 93.345) (end 220.98 91.44) (width 2) (layer B.Cu) (net 16))
-  (segment (start 219.075 93.345) (end 215.9 93.345) (width 2) (layer F.Cu) (net 16))
-  (segment (start 220.98 91.44) (end 219.075 93.345) (width 2) (layer F.Cu) (net 16))
-  (segment (start 220.98 83.82) (end 220.98 91.44) (width 2) (layer F.Cu) (net 16))
-  (segment (start 209.55 79.375) (end 216.535 79.375) (width 2) (layer F.Cu) (net 16))
-  (segment (start 216.535 79.375) (end 220.98 83.82) (width 2) (layer F.Cu) (net 16))
   (segment (start 215.9 101.275) (end 215.9 98.425) (width 2) (layer B.Cu) (net 17))
   (segment (start 215.9 103.965) (end 215.9 101.275) (width 2) (layer B.Cu) (net 17))
@@
     (connect_pads (clearance 0.254))
     (min_thickness 0.254)
-    (fill yes (arc_segments 16) (thermal_gap 0.508) (thermal_bridge_width 0.508) (smoothing fillet) (radius 0.254))
+    (fill yes (arc_segments 16) (thermal_gap 0.508) (thermal_bridge_width 0.508) (smoothing fillet) (radius 0.5))
     (polygon
       (pts
@@
     (connect_pads yes (clearance 0.254))
     (min_thickness 0.254)
-    (fill yes (arc_segments 16) (thermal_gap 0.508) (thermal_bridge_width 0.508))
+    (fill yes (arc_segments 16) (thermal_gap 0.508) (thermal_bridge_width 0.508) (smoothing fillet) (radius 0.5))
     (polygon
       (pts
@@
       )
     )
+  )
+  (zone (net 2) (net_name /12V_Out) (layer B.Cu) (hatch edge 0.508)
+    (priority 1)
+    (connect_pads (clearance 0.254))
+    (min_thickness 0.254)
+    (fill yes (arc_segments 32) (thermal_gap 0.508) (thermal_bridge_width 0.508) (smoothing fillet) (radius 0.5))
+    (polygon
+      (pts
+        (xy 212.725 83.693) (xy 212.725 92.075) (xy 217.424 92.075) (xy 217.424 83.693)
+      )
+    )
+  )
+  (zone (net 2) (net_name /12V_Out) (layer F.Cu) (hatch edge 0.508)
+    (priority 1)
+    (connect_pads (clearance 0.254))
+    (min_thickness 0.254)
+    (fill yes (arc_segments 32) (thermal_gap 0.508) (thermal_bridge_width 0.508) (smoothing fillet) (radius 0.5))
+    (polygon
+      (pts
+        (xy 212.725 83.693) (xy 212.725 92.075) (xy 217.424 92.075) (xy 217.424 83.693)
+      )
+    )
